File: stepper_sc/stepper_sc.kicad_sch (KiCad schematic)
At the start: 24 parts, among them J1 PWR_24V, J10 BUZZ, J11 Black_Pill_front, J12 Black_Pill_back, J2 PUL, J3 DIR, J4 ES_L, J5 ES_R, J6 JOGL, J7 JOGR, J8 STEPL, J9 STEPR, Q1 BC547, Q2 BC547, U1 78M05

Commit message: Change C1 and C3 footprints to SMD electrolytic CP_Elec_8x6.2
Both 100µF caps replaced: Capacitor_THT:CP_Radial_D8.0mm_P3.50mm
→ Capacitor_SMD:CP_Elec_8x6.2

Schematic edited directly (kicad-sch-api strips lib_symbols on save —
do not use it for footprint changes on this schematic).
PCB updated via F8 Update PCB from Schematic.

Co-Authored-By: Claude Sonnet 4.6 <noreply@anthropic.com>
Parts:
- C1, C3: footprint Capacitor_THT:CP_Radial_D8.0mm_P3.50mm -> Capacitor_SMD:CP_Elec_8x6.2
Changed lines of the file:
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@@
 			)
 		)
-		(property "Footprint" "Capacitor_THT:CP_Radial_D8.0mm_P3.50mm"
+		(property "Footprint" "Capacitor_SMD:CP_Elec_8x6.2"
 			(at 61.9252 34.29 0.0000)
 			(effects
@@
 			)
 		)
-		(property "Footprint" "Capacitor_THT:CP_Radial_D8.0mm_P3.50mm"
+		(property "Footprint" "Capacitor_SMD:CP_Elec_8x6.2"
 			(at 117.8052 34.29 0.0000)
 			(effects

Commit message: PCB: swap C1/C3→CP_Elec_8x6.2 SMD, Q1/Q2→SOT-23 SMD; assign pad nets
- C1, C3: Capacitor_THT:CP_Radial_D8.0mm_P3.50mm → Capacitor_SMD:CP_Elec_8x6.2
- Q1, Q2: Package_TO_SOT_THT:TO-92_Inline → Package_TO_SOT_SMD:SOT-23
- Q1 pads: pad1(B)→Net-(Q1-PadB), pad2(E)→GND, pad3(C)→Net-(J2-Pin_2)
- Q2 pads: pad1(B)→Net-(Q2-PadB), pad2(E)→GND, pad3(C)→Net-(J3-Pin_2)
- Re-placed all 24 footprints after footprint swap

Co-Authored-By: Claude Sonnet 4.6 <noreply@anthropic.com>
Parts:
- Q1, Q2: footprint Package_TO_SOT_THT:TO-92_Inline -> Package_TO_SOT_SMD:SOT-23
Changed lines of the file:
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@@
 			)
 		)
-		(property "Footprint" "Package_TO_SOT_THT:TO-92_Inline"
+		(property "Footprint" "Package_TO_SOT_SMD:SOT-23"
 			(at 81.28 91.44 0.0000)
 			(effects
@@
 			)
 		)
-		(property "Footprint" "Package_TO_SOT_THT:TO-92_Inline"
+		(property "Footprint" "Package_TO_SOT_SMD:SOT-23"
 			(at 81.28 123.19 0.0000)
 			(effects
